Commit message: Split launch per behaviour, restore goal navigation, fix goal overshoot
Separate the two behaviours into their own launch files over a shared
simulation bring-up, and correct two ways the robot drove past its goal.

- Add simulation.launch.py (Gazebo, spawn, controllers, RViz) and layer
  geofence.launch.py and goal_navigation.launch.py on top of it. The
  simulation file can also be run alone for manual driving.
- Restore Week 1's goal navigation as a second 'behavior' mode on the
  same node rather than a forked copy, so both modes share one avoidance
  implementation. goal_x/goal_y are overridable at launch.
- Turn in place until within heading_tolerance_deg of the target bearing,
  then drive straight, instead of steering continuously the whole way. A
  pivot scrubs more per degree, but it minimises total rotation, and
  rotation is where the odometry error comes from: a straight 10 m run
  finished 0.01 m from ground truth, while a 5 m run containing one
  avoidance turn finished 2.3 m out.
- Cap forward speed by proximity to the goal in every state, not only
  while goal-seeking. CLEARING drives at full speed and returns before
  the goal-navigation branch runs, so a goal inside its clearing run was
  crossed at 1.0 m/s and overshot by the 0.25 m stopping distance.
- Check goal arrival ahead of the avoidance states, which return early,
  so CLEARING no longer drives its full clearing_distance past a goal.
- Wrap the xacro output in ParameterValue(value_type=str). Without it
  launch parses the URDF as YAML, and any "word:" sequence in the XML
  aborts the launch after Gazebo has already started, leaving an empty
  world with no robot in it.
- Give the wheels a cylinder's inertia (axial 0.01125, transverse 0.0075)
  instead of 0.01 on all three axes, which describes a sphere.
- Lower wheel friction to mu 0.3.

Co-Authored-By: Claude Opus 5 <noreply@anthropic.com>

File: urdf/egrobots_rover.urdf.xacro (robot description, xacro)
@@ -42,5 +42,9 @@
     <inertial>
       <mass value="1.0"/>
-      <inertia ixx="0.01" ixy="0.0" ixz="0.0" iyy="0.01" iyz="0.0" izz="0.01"/>
+      <!-- Solid cylinder r=0.15, L=0.15, m=1.0, spinning about Y (the joint axis).
+           Axial term    m*r^2/2           = 0.01125  (iyy)
+           Transverse    m*(3r^2 + L^2)/12 = 0.0075   (ixx, izz)
+           Previously 0.01 on all three axes, which describes a sphere, not a wheel. -->
+      <inertia ixx="0.0075" ixy="0.0" ixz="0.0" iyy="0.01125" iyz="0.0" izz="0.0075"/>
     </inertial>
   </link>
@@ -67,5 +71,9 @@
     <inertial>
       <mass value="1.0"/>
-      <inertia ixx="0.01" ixy="0.0" ixz="0.0" iyy="0.01" iyz="0.0" izz="0.01"/>
+      <!-- Solid cylinder r=0.15, L=0.15, m=1.0, spinning about Y (the joint axis).
+           Axial term    m*r^2/2           = 0.01125  (iyy)
+           Transverse    m*(3r^2 + L^2)/12 = 0.0075   (ixx, izz)
+           Previously 0.01 on all three axes, which describes a sphere, not a wheel. -->
+      <inertia ixx="0.0075" ixy="0.0" ixz="0.0" iyy="0.01125" iyz="0.0" izz="0.0075"/>
     </inertial>
   </link>
@@ -92,5 +100,9 @@
     <inertial>
       <mass value="1.0"/>
-      <inertia ixx="0.01" ixy="0.0" ixz="0.0" iyy="0.01" iyz="0.0" izz="0.01"/>
+      <!-- Solid cylinder r=0.15, L=0.15, m=1.0, spinning about Y (the joint axis).
+           Axial term    m*r^2/2           = 0.01125  (iyy)
+           Transverse    m*(3r^2 + L^2)/12 = 0.0075   (ixx, izz)
+           Previously 0.01 on all three axes, which describes a sphere, not a wheel. -->
+      <inertia ixx="0.0075" ixy="0.0" ixz="0.0" iyy="0.01125" iyz="0.0" izz="0.0075"/>
     </inertial>
   </link>
@@ -117,5 +129,9 @@
     <inertial>
       <mass value="1.0"/>
-      <inertia ixx="0.01" ixy="0.0" ixz="0.0" iyy="0.01" iyz="0.0" izz="0.01"/>
+      <!-- Solid cylinder r=0.15, L=0.15, m=1.0, spinning about Y (the joint axis).
+           Axial term    m*r^2/2           = 0.01125  (iyy)
+           Transverse    m*(3r^2 + L^2)/12 = 0.0075   (ixx, izz)
+           Previously 0.01 on all three axes, which describes a sphere, not a wheel. -->
+      <inertia ixx="0.0075" ixy="0.0" ixz="0.0" iyy="0.01125" iyz="0.0" izz="0.0075"/>
     </inertial>
   </link>
@@ -179,21 +195,21 @@
   <gazebo reference="wheel_front_left">
     <material>Gazebo/Black</material>
-    <mu1>0.6</mu1>
-    <mu2>0.6</mu2>
+    <mu1>0.3</mu1>
+    <mu2>0.3</mu2>
   </gazebo>
   <gazebo reference="wheel_front_right">
     <material>Gazebo/Black</material>
-    <mu1>0.6</mu1>
-    <mu2>0.6</mu2>
+    <mu1>0.3</mu1>
+    <mu2>0.3</mu2>
   </gazebo>
   <gazebo reference="wheel_rear_left">
     <material>Gazebo/Black</material>
-    <mu1>0.6</mu1>
-    <mu2>0.6</mu2>
+    <mu1>0.3</mu1>
+    <mu2>0.3</mu2>
   </gazebo>
   <gazebo reference="wheel_rear_right">
     <material>Gazebo/Black</material>
-    <mu1>0.6</mu1>
-    <mu2>0.6</mu2>
+    <mu1>0.3</mu1>
+    <mu2>0.3</mu2>
   </gazebo>
   <gazebo reference="mast">

Commit message: Fuse IMU with wheel odometry via an EKF to correct heading drift
Wheel encoders cannot observe the sideways scrub a skid-steer needs to
turn, so heading was the dominant source of position error. Add an IMU
and let robot_localization fuse the two.

- Add an imu_link to the URDF with libgazebo_ros_imu_sensor publishing
  /imu/data at 100 Hz, rigidly fixed to the chassis near the centre of
  rotation, with gaussian noise on yaw rate so it is not a perfect
  oracle reading ground truth.
- Add config/ekf.yaml taking only forward velocity from the wheels and
  only yaw and yaw rate from the IMU. Measured on this rover, wheel
  odometry tracks distance at 98-102% over 10 m but reports 85 deg of
  rotation for 63 deg of real turn, so each sensor supplies the quantity
  it measures well.
- Exclude the wheels' yaw entirely rather than down-weighting it. A
  Kalman filter averages out noise but not bias, and skid-steer wheel
  yaw is biased by a near-constant factor, which would drag the estimate
  toward the wrong answer.
- Set enable_odom_tf: false so ekf_filter_node owns odom -> base_link.
  The controller still publishes /diff_drive_controller/odom as an input
  to the filter; two publishers of one transform would fight.
- Declare the robot_localization dependency, which rosdep would
  otherwise not install on a clean machine.

obstacle_avoider_node is unchanged: it asks TF2 for odom -> base_link and
does not care which node answers.

Measured on the same obstacle-avoidance run to goal (5.0, 0.0):
wheel odometry alone reported (4.87, 0.08) while ground truth was
(7.19, 0.73), a 2.3 m error. With the EKF it reported (4.97, -0.14)
against a true (5.07, -0.19) — 0.09 m.

Drift is reduced, not eliminated: dead reckoning still has no absolute
reference, and a simulated IMU lacks the gyro bias drift of a real one.
README section 7 now describes what remains and why LiDAR localization
would be the next step.

Co-Authored-By: Claude Opus 5 <noreply@anthropic.com>

File: urdf/egrobots_rover.urdf.xacro (robot description, xacro)
@@ -190,4 +190,18 @@
     <origin xyz="0 0 0" rpy="0 0 0"/>
   </joint>
+  <!-- IMU, mounted on the chassis. Its yaw measurement is independent of the
+       wheels, so it is unaffected by the sideways scrub that corrupts wheel
+       odometry on a skid-steer platform. -->
+  <link name="imu_link">
+    <inertial>
+      <mass value="0.01"/>
+      <inertia ixx="1e-6" ixy="0.0" ixz="0.0" iyy="1e-6" iyz="0.0" izz="1e-6"/>
+    </inertial>
+  </link>
+  <joint name="imu_joint" type="fixed">
+    <parent link="base_link"/>
+    <child link="imu_link"/>
+    <origin xyz="0 0 0.1" rpy="0 0 0"/>
+  </joint>
   <gazebo reference="base_link">
     <material>Gazebo/DarkGrey</material>
@@ -218,4 +232,30 @@
   <gazebo reference="sensor_mount">
     <material>Gazebo/Black</material>
+  </gazebo>
+  <gazebo reference="imu_link">
+    <gravity>true</gravity>
+    <sensor name="imu_sensor" type="imu">
+      <always_on>true</always_on>
+      <update_rate>100</update_rate>
+      <visualize>false</visualize>
+      <plugin name="imu_plugin" filename="libgazebo_ros_imu_sensor.so">
+        <ros>
+          <namespace>/</namespace>
+          <remapping>~/out:=imu/data</remapping>
+        </ros>
+        <frame_name>imu_link</frame_name>
+        <initial_orientation_as_reference>false</initial_orientation_as_reference>
+      </plugin>
+      <imu>
+        <angular_velocity>
+          <z>
+            <noise type="gaussian">
+              <mean>0.0</mean>
+              <stddev>2e-4</stddev>
+            </noise>
+          </z>
+        </angular_velocity>
+      </imu>
+    </sensor>
   </gazebo>
   <gazebo>
